File: _autosave-Banc d'essais.kicad_pcb (KiCad board)
At the start: 2 copper layers, 3 parts, among them U1 MCP4431-xxxx-ST

Commit message: modification + finalisation du PCB et du schéma
Parts:
- removed U1: MCP4431-xxxx-ST, Package_SO:TSSOP-20_4.4x6.5mm_P0.65mm
- moved Ecran1 52.3 mm to (139.5, 55.1)
- moved A1 30.2 mm to (130.7, 49.7)
Routing:
- net Net-(A1-+5V): track 0.00 -> 41.0 mm
- net Net-(Ecran1-K): track 0.00 -> 22.2 mm
Other:
- board text added: "BTS CIEL2 Conçu par Enzo Lethiais"
