File: Banc d'essais.kicad_sch (KiCad schematic)
At the start: 0 parts

Commit message: edrthgnb,fd j;gbdukjfth,cnv
Parts:
- added A1: Arduino_UNO_R3, Module:Arduino_UNO_R3, symbol MCU_Module:Arduino_UNO_R3
- added Ecran1: ~, banc_d'essais:Sans titre, symbol banc_d'essais:EcranLCD
- added U1: MCP4431-xxxx-ST, Package_SO:TSSOP-20_4.4x6.5mm_P0.65mm, symbol Potentiometer_Digital:MCP4431-xxxx-ST
Connections:
- new net: A1.3 (~{RESET}), A1.4 (3V3), A1.5 (+5V), Ecran1.1 (VDD), Ecran1.12 (DB5), Ecran1.13 (DB6), U1.11 (P0A)
- new net: A1.2 (IOREF), Ecran1.14 (DB7)
- new net: Ecran1.3 (V0), U1.12 (P0W)
- new net: A1.12 (A3), Ecran1.4 (RS)
- new net: A1.11 (A2), Ecran1.6 (E)
- new net Earth: Ecran1.16 (K), Ecran1.2 (VSS), Ecran1.5 (R/W), U1.13 (P0B)

Commit message: modification + finalisation du PCB et du schéma
Parts:
- added TP1, TP2: TestPoint, symbol Connector:TestPoint
Connections:
- net Earth: now also Ecran1.3 (V0), U1.12 (P0W), TP2.1
- net at A1.3 (~{RESET}), A1.4 (3V3), A1.5 (+5V)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: now also TP1.1
Other:
- note added: "Schéma du Banc d'essais pour écran LCD"
- moved on the sheet: A1, Ecran1, U1A

Commit message: Réarrangement des dossiers
Parts:
- added TP3: TestPoint, symbol Connector:TestPoint
Connections:
- net at A1.2 (IOREF), Ecran1.14 (DB7): now also TP3.1
Changed lines of the file:
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@@
+	)
+	(junction
+		(at 130.81 73.66)
+		(diameter 0)
+		(color 0 0 0 0)
 	)
 	(junction
@@
 	(wire
 		(pts
+			(xy 130.81 73.66) (xy 187.96 73.66)
+		)
+		(stroke
+			(width 0)
+			(type default)
+		)
+	)
+	(wire
+		(pts
 			(xy 149.86 97.79) (xy 157.48 97.79)
 		)
@@
 	(wire
 		(pts
-			(xy 123.19 73.66) (xy 187.96 73.66)
+			(xy 123.19 73.66) (xy 130.81 73.66)
 		)
 		(stroke
@@
 		(pts
 			(xy 148.59 78.74) (xy 148.59 81.28)
+		)
+		(stroke
+			(width 0)
+			(type default)
+		)
+	)
+	(wire
+		(pts
+			(xy 130.81 73.66) (xy 130.81 78.74)
 		)
 		(stroke
@@
 					(unit 1)
 				)
+			)
+		)
+	)
+	(symbol
+		(lib_id "Connector:TestPoint")
+		(at 130.81 78.74 180)
+		(unit 1)
+		(exclude_from_sim no)
+		(in_bom yes)
+		(on_board yes)
+		(dnp no)
+		(fields_autoplaced yes)
+		(property "Reference" "TP3"
+			(at 133.35 80.7719 0)
+			(effects
+				(font
+					(size 1.27 1.27)
+				)
+				(justify right)
+			)
+		)
+		(property "Value" "TestPoint"
+			(at 133.35 83.3119 0)
+			(effects
+				(font
+					(size 1.27 1.27)
+				)
+				(justify right)
+			)
+		)
+		(property "Footprint" ""
+			(at 125.73 78.74 0)
+			(effects
+				(font
+					(size 1.27 1.27)
+				)
+				(hide yes)
+			)
+		)
+		(property "Datasheet" "~"
+			(at 125.73 78.74 0)
+			(effects
+				(font
+					(size 1.27 1.27)
+				)
+				(hide yes)
+			)
+		)
+		(property "Description" "test point"
+			(at 130.81 78.74 0)
+			(effects
+				(font
+					(size 1.27 1.27)
+				)
+				(hide yes)
+			)
+		)
+		(pin "1"
+		)
+		(instances
+			(project ""
+				(path "/137ff572-d30e-44d7-a0ef-739ddc99a077"
+					(reference "TP3")
+					(unit 1)
+				)
