File: PCB+Schéma/Banc d'essais.kicad_pcb (KiCad board)
At the start: 2 copper layers, 2 parts

Commit message: mise a jours
Parts:
- added RV1: R_Potentiometer, Potentiometer_THT:Potentiometer_ACP_CA6-H2,5_Horizontal, F.Cu at (145.2, 118.0)
Connections:
- A1 pad 11: unconnected-(A1-A2-Pad11) -> Net-(A1-A2)
- A1 pad 12: unconnected-(A1-A3-Pad12) -> Net-(A1-A3)
- A1 pad 2: unconnected-(A1-IOREF-Pad2) -> Net-(A1-IOREF)
- A1 pad 3: unconnected-(A1-~{RESET}-Pad3) -> Net-(A1-+5V)
- A1 pad 4: unconnected-(A1-3V3-Pad4) -> Net-(A1-+5V)
- Ecran1 pad 12: unconnected-(Ecran1-DB5-Pad12) -> Net-(A1-+5V)
- Ecran1 pad 13: unconnected-(Ecran1-DB6-Pad13) -> Net-(A1-+5V)
- Ecran1 pad 14: unconnected-(Ecran1-DB7-Pad14) -> Net-(A1-IOREF)
- Ecran1 pad 16: Net-(Ecran1-K) -> Earth
- Ecran1 pad 2: Net-(Ecran1-K) -> Earth
- Ecran1 pad 3: Net-(Ecran1-V0) -> Earth
- Ecran1 pad 4: unconnected-(Ecran1-RS-Pad4) -> Net-(A1-A3)
- Ecran1 pad 5: Net-(Ecran1-K) -> Earth
- Ecran1 pad 6: unconnected-(Ecran1-E-Pad6) -> Net-(A1-A2)
Routing:
- net Earth: track 0.00 -> 72.9 mm, vias 0 -> 4
- net Net-(A1-+5V): track 41.0 -> 94.8 mm
- net Net-(A1-A3): track 0.00 -> 38.7 mm, vias 0 -> 1
- net Net-(A1-A2): track 0.00 -> 29.5 mm
- net Net-(Ecran1-K): track 22.2 -> 0.00 mm
- net Net-(A1-IOREF): track 0.00 -> 16.2 mm
